File: AS3364 DG412 bus mixer v1.0.sch (EAGLE design)
At the start: 122 parts, among them IC1 PCA9539PW, IC10 DG412-J, IC11 DG412-J, IC14 TL074JT, IC2 TL074JT, IC3 TL072JT, IC4 TL074JT, IC6 TL072JT, IC8 DG412-J, IC9 DG412-J

Commit message: Added sum a and b to output pins
Parts:
- removed SV2, SV34, SV35: (no value), joakim:MA08-1JP
- added SV1, SV3, SV4: (no value), joakim:MA08-1JP
Connections:
- removed net LPF_IN_100K_MIX: R70.2, R72.2, SV35.2
- removed net SVF_IN_100K_MIX: R69.2, R71.2, SV35.1
- new net OUT_A_100K_MIX: R69.2, R71.2, SV4.2
- new net OUT_B_100K_MIX: R70.2, R72.2, SV4.3
- net +12V: now also SV4.6; no longer SV35.5
- net -12V: now also SV4.8; no longer SV35.7
- net CV1: now also SV33.8; no longer SV34.1
- net CV2: now also SV1.1; no longer SV34.2
- net CV3: now also SV1.2; no longer SV34.3
- net CV4: now also SV1.3; no longer SV34.4
- net CV5: now also SV3.3; no longer SV2.2
- net CV6: now also SV3.4; no longer SV2.3
- net CV7: now also SV3.5; no longer SV2.4
- net CV8: now also SV3.6; no longer SV2.5
- net CV_A_DRY: now also SV1.8; no longer SV34.7
- net CV_A_WET: now also SV4.4; no longer SV35.3
- net CV_B_DRY: now also SV4.1; no longer SV34.8
- net CV_B_WET: now also SV4.5; no longer SV35.4
- net GND: now also SV4.7; no longer SV35.6
- net IN1: now also SV33.6; no longer SV33.7
- net IN2: now also SV33.7; no longer SV33.8
- net IN3: now also SV1.4; no longer SV34.5
- net IN4: now also SV1.5; no longer SV34.6
- net IN5: now also SV3.1; no longer SV35.8
- net IN6: now also SV3.2; no longer SV2.1
- net IN7: now also SV3.7; no longer SV2.6
- net IN8: now also SV3.8; no longer SV2.7
- net SUM_A: now also SV1.6
- net SUM_B: now also SV1.7
Other:
- note added: "TODO: CHECK PHASE OF FX SIGNAL!"
- note removed: "TODO: Clipping detector?"
- note removed: "TODO: DIST HAR EGEN AMP SE OM VI TRENGER DENNE OG "VANLIG" Hvis vi kombinerer så kan vi antakelig kombinere siste celle her med de tre vi trenger for VCO"

Commit message: New version with inverted vcas on inputs
Parts:
- added C24, C25, C26, C27: 33pF, joakim:C-EU-J
Connections:
- net BUS_A: now also C24.1
- net BUS_B: now also C25.1
- net BUS_FX_A: now also C26.1
- net BUS_FX_B: now also C27.1
- net CON1: now also IC3B.-IN; no longer IC3B.+IN
- net CON2: now also IC3A.-IN; no longer IC3A.+IN
- net CON3: now also IC14B.-IN; no longer IC14B.+IN
- net CON4: now also IC14C.-IN; no longer IC14C.+IN
- net CON5: now also IC2A.-IN; no longer IC2A.+IN
- net CON6: now also IC2D.-IN; no longer IC2D.+IN
- net CON7: now also IC6B.-IN; no longer IC6B.+IN
- net CON8: now also IC6A.-IN; no longer IC6A.+IN
- net GND: now also IC14B.+IN, IC14C.+IN, IC2A.+IN, IC2D.+IN, IC3A.+IN, IC3B.+IN, IC6A.+IN, IC6B.+IN; no longer R41.1, R42.1, R43.1, R44.1, R45.1, R46.1, R47.1, R48.1
- net OUT1: now also R44.1; no longer IC3B.-IN
- net OUT2: now also R41.1; no longer IC3A.-IN
- net OUT3: now also R43.1; no longer IC14B.-IN
- net OUT4: now also R42.1; no longer IC14C.-IN
- net OUT5: now also R48.1; no longer IC2A.-IN
- net OUT6: now also R45.1; no longer IC2D.-IN
- net OUT7: now also R47.1; no longer IC6B.-IN
- net OUT8: now also R46.1; no longer IC6A.-IN
- net SUM_A: now also C24.2
- net SUM_B: now also C25.2
- net SUM_FX_A: now also C26.2
- net SUM_FX_B: now also C27.2
Other:
- note added: "100kHz LPF"
- note removed: "TODO: CHECK PHASE OF FX SIGNAL!"
- moved on the sheet: C23, IC1, IC4A, IC4C, R1, R41, R42, R43, R44, R45, R46, R47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

Commit message: Fixed pin labeling
Parts:
- C13, C14, C15: device rcl:C-EUC0402 -> joakim:C-EU-J
Changed lines of the file:
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@@
 <part name="IC3" library="joakim" deviceset="TL072J" device="T" value="TL072JT"/>
 <part name="C18" library="rcl" library_urn="urn:adsk.eagle:library:334" deviceset="C-EU" device="C0402" package3d_urn="urn:adsk.eagle:package:23626/2" value="100nF"/>
-<part name="C13" library="rcl" library_urn="urn:adsk.eagle:library:334" deviceset="C-EU" device="C0402" package3d_urn="urn:adsk.eagle:package:23626/2" value="5nF"/>
+<part name="C13" library="joakim" deviceset="C-EU-J" device="" package3d_urn="urn:adsk.eagle:package:23547/3" value="5nF"/>
 <part name="GND9" library="supply1" library_urn="urn:adsk.eagle:library:371" deviceset="GND" device=""/>
 <part name="DA2" library="joakim" deviceset="AS3364" device="D"/>
@@
 <part name="GND17" library="supply1" library_urn="urn:adsk.eagle:library:371" deviceset="GND" device=""/>
 <part name="GND18" library="supply1" library_urn="urn:adsk.eagle:library:371" deviceset="GND" device=""/>
-<part name="C14" library="rcl" library_urn="urn:adsk.eagle:library:334" deviceset="C-EU" device="C0402" package3d_urn="urn:adsk.eagle:package:23626/2" value="5nF"/>
+<part name="C14" library="joakim" deviceset="C-EU-J" device="" package3d_urn="urn:adsk.eagle:package:23547/3" value="5nF"/>
 <part name="GND19" library="supply1" library_urn="urn:adsk.eagle:library:371" deviceset="GND" device=""/>
 <part name="DA3" library="joakim" deviceset="AS3364" device="D"/>
@@
 <part name="GND37" library="supply1" library_urn="urn:adsk.eagle:library:371" deviceset="GND" device=""/>
 <part name="IC6" library="joakim" deviceset="TL072J" device="T" value="TL072JT"/>
-<part name="C15" library="rcl" library_urn="urn:adsk.eagle:library:334" deviceset="C-EU" device="C0402" package3d_urn="urn:adsk.eagle:package:23626/2" value="5nF"/>
+<part name="C15" library="joakim" deviceset="C-EU-J" device="" package3d_urn="urn:adsk.eagle:package:23547/3" value="5nF"/>
 <part name="GND38" library="supply1" library_urn="urn:adsk.eagle:library:371" deviceset="GND" device=""/>
 <part name="DA1" library="joakim" deviceset="AS3364" device="D"/>

Commit message: TODO about needing to invert output
Other:
- note added: "TODO: PGA manglende summer på filter output så kan man ikke ha to LPF. Det må fikses. Ha inverted output og summer enten her eller eksternt"
Changed lines of the file:
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@@
 <text x="-91.44" y="55.88" size="1.778" layer="91">C2833322 8p</text>
 <text x="264.16" y="38.1" size="1.778" layer="97">100kHz LPF</text>
+<text x="-17.78" y="124.46" size="6.4516" layer="91">TODO:
+PGA manglende summer
+på filter output
+så kan man ikke ha to
+LPF. Det må fikses.
+Ha inverted output
+og summer enten her
+eller eksternt</text>
 </plain>
 <instances>
