File: attic/AS3364 DG412 bus mixer v1.0 copy.sch (EAGLE design)
At the start: 121 parts, among them IC1 PCA9539PW, IC10 DG412-J, IC11 DG412-J, IC2 TL074JT, IC3 TL072JT, IC4 TL074JT, IC5 TL072JT, IC6 TL072JT, IC8 DG412-J, IC9 DG412-J, X1 MA17-1JP

Commit message: Cleanup
Parts:
- removed C24, C25, C26, C27: 33pF, joakim:C-EU-J
- removed IC5: TL072JT, joakim:TL072JT
- removed U$2: MA16-1JP, joakim:MA16-1JP
- removed X1: MA17-1JP, joakim:MA17-1JP
- added IC14: TL074JT, joakim:TL074JT
- added R70, R71, R72: 100k, rcl:R-EU_R0402
- added SV1, SV10, SV11, SV12, SV13, SV14, SV15, SV16, SV17, SV18, SV19, SV2, SV20, SV21, SV22, SV23, SV24, SV25, SV26, SV27, SV28, SV29, SV3, SV30, SV31, SV32, SV4, SV5, SV6, SV7, SV8, SV9: (no value), joakim:MA01-1JP
- C13, C14, C15: device joakim:C-EU-J -> rcl:C-EUC0402
- R69: value 47k -> 100k
- R77: value 47k -> 105k
- R78: value 33k -> 75k
Connections:
- removed net N$17: DA1G$1.OUT1, IC2C.+IN, R51.1
- removed net N$18: DA1G$1.OUT4, IC2B.+IN, R49.1
- removed net N$19: DA3G$1.OUT3, IC6B.+IN, R47.1
- removed net N$4: DA3G$1.OUT2, IC6A.+IN, R46.1
- removed net N$6: DA1G$1.OUT2, IC2C.-IN, R50.2, R69.1
- removed net SVF_CHAIN: R69.2, X1.17
- new net CON7: DA3G$1.OUT3, IC6B.+IN, R47.2
- new net CON8: DA3G$1.OUT2, IC6A.+IN, R46.2
- new net CON_O2: DA1G$1.OUT1, IC14D.+IN, R49.2
- new net CON_O3: DA1G$1.OUT3, IC2B.+IN, R51.2
- new net CON_O4: DA1G$1.OUT2, IC2C.+IN, R50.2
- new net LPF_IN_100K_MIX: R70.2, R72.2, SV20.1
- new net OUT_FX_A: IC2B.-IN, IC2B.OUT, R71.1
- new net OUT_FX_B: IC2C.-IN, IC2C.OUT, R72.1
- new net SVF_IN_100K_MIX: R69.2, R71.2, SV19.1
- net !RST: now also SV6.1; no longer X1.5
- net +12V: now also IC14P.V+, SV21.1; no longer IC5P.V+, U$2.6
- net +3V3: now also SV2.1; no longer X1.1
- net -12V: now also IC14P.V-, SV31.1; no longer IC5P.V-, U$2.8
- net BUS_A: no longer C24.1
- net BUS_B: no longer C25.1
- net BUS_FX_A: no longer C26.1
- net BUS_FX_B: no longer C27.1
- net CON1: now also IC3B.+IN; no longer IC3B.-IN
- net CON2: now also IC3A.+IN; no longer IC3A.-IN
- net CON3: now also IC14B.+IN; no longer IC5B.-IN
- net CON4: now also IC14C.+IN; no longer IC5A.-IN
- net CON5: now also IC2A.+IN; no longer IC2A.-IN
- net CON6: now also IC2D.+IN; no longer IC2D.-IN
- net CON_O1: now also DA1G$1.OUT4, IC14A.+IN; no longer DA1G$1.OUT3, IC2B.-IN
- net CV1: now also SV11.1; no longer X1.8
- net CV2: now also SV12.1; no longer X1.9
- net CV3: now also SV13.1; no longer X1.10
- net CV4: now also SV14.1; no longer X1.11
- net CV5: now also SV27.1; no longer U$2.11
- net CV6: now also SV28.1; no longer U$2.12
- net CV7: now also SV29.1; no longer U$2.13
- net CV8: now also SV30.1; no longer U$2.14
- net CV_A_DRY: now also SV15.1; no longer X1.16
- net CV_A_WET: now also SV16.1; no longer U$2.4
- net CV_B_DRY: now also SV17.1; no longer U$2.1
- net CV_B_WET: now also SV18.1; no longer U$2.5
- net DGND: now also SV5.1; no longer X1.4
- net GND: now also R41.1, R42.1, R43.1, R44.1, R45.1, R46.1, R47.1, R48.1, R49.1, R50.1, R51.1, R52.1, SV22.1; no longer IC2A.+IN, IC2D.+IN, IC3A.+IN, IC3B.+IN, IC5A.+IN, IC5B.+IN, R46.2, R47.2, R49.2, R51.2, U$2.7
- net IN1: now also SV7.1; no longer X1.6
- net IN2: now also SV8.1; no longer X1.7
- net IN3: now also SV9.1; no longer X1.12
- net IN4: now also SV10.1; no longer X1.13
- net IN5: now also SV23.1; no longer U$2.9
- net IN6: now also SV24.1; no longer U$2.10
- net IN7: now also SV25.1; no longer U$2.15
- net IN8: now also SV26.1; no longer U$2.16
- net OUT1: now also IC3B.-IN; no longer R44.1
- net OUT2: now also IC3A.-IN; no longer R41.1
- net OUT3: now also IC14B.-IN, IC14B.OUT; no longer IC5B.OUT, R43.1
- net OUT4: now also IC14C.-IN, IC14C.OUT; no longer IC5A.OUT, R42.1
- net OUT5: now also IC2A.-IN; no longer R48.1
- net OUT6: now also IC2D.-IN; no longer R45.1
- net OUT_A: now also IC14A.-IN, IC14A.OUT, R69.1; no longer IC2B.OUT, R52.1, U$2.2
- net OUT_B: now also IC14D.-IN, IC14D.OUT, R70.1; no longer IC2C.OUT, R50.1, U$2.3
- net SCL: now also SV4.1; no longer X1.3
- net SDA: now also SV3.1; no longer X1.2
- net SUM_A: no longer C24.2, X1.14
- net SUM_B: no longer C25.2, X1.15
- net SUM_FX_A: no longer C26.2
- net SUM_FX_B: no longer C27.2
Other:
- note added: "NB: Mixed by op amp externally"
- note added: "TODO: Clipping detector?"
- note added: "TODO: DIST HAR EGEN AMP SE OM VI TRENGER DENNE OG "VANLIG" Hvis vi kombinerer så kan vi antakelig kombinere siste celle her med de tre vi trenger for VCO"
- note removed: "1.2: 2 x 16p instead of 1 x 32p 1.3: ext input to output B, to add SVF output, mixed here to get clipping BEFORE Juno filter"
- note removed: "100kHz LPF"
- note removed: "C2833322 8p"
- note removed: "Funker finfint!"
- note removed: "Inverts FX but not Dry so output is in phase"
- note removed: "NB: FX is inv here"
- note removed: "NB: FX is non-inv here"
- note removed: "NB: SVF Chain is inverting!"
- moved on the sheet: C23, IC1, IC2B, IC4A, IC4C, R1, R41, R42, R43, R44, R45, R46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
