File: Bus_Mixer/Angle board.sch (EAGLE design)
At the start: 4 parts

Commit message: v1.0 ready for production
Connections:
- removed net N$29: U$2.4, U$4.13
- removed net N$7: U$1.7, U$3.10
- new net AGND: U$1.7, U$2.4, U$3.10, U$4.13
Other:
- moved on the sheet: U$1, U$2
