File: Bus_Mixer/slim bus mixer v1-4-layer.sch (EAGLE design)
At the start: 148 parts, among them IC1 PCA9539PW, IC10 DG412-JT, IC11 DG412-JT, IC2 TL074JT, IC3 TL072JT, IC4 TL074JT, IC6 TL072JT, IC7 TL074JT, IC8 DG412-JT, IC9 DG412-JT

Commit message: moving to single line for switches + control
Parts:
- IC10, IC11, IC8, IC9: value DG412-JT -> DG412-JS; device joakim:DG412-JT -> joakim:DG412-JS
Other:
- note added: "SOIC16 version available as Pre-order at JLCPCB, half price or less than TSSOP"
Changed lines of the file:
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@@
 <part name="R66" library="rcl" library_urn="urn:adsk.eagle:library:334" deviceset="R-EU_" device="R0402" package3d_urn="urn:adsk.eagle:package:23547/3" value="47k"/>
 <part name="R68" library="rcl" library_urn="urn:adsk.eagle:library:334" deviceset="R-EU_" device="R0402" package3d_urn="urn:adsk.eagle:package:23547/3" value="47k"/>
-<part name="IC8" library="joakim" deviceset="DG412-J" device="T" value="DG412-JT"/>
-<part name="IC9" library="joakim" deviceset="DG412-J" device="T" value="DG412-JT"/>
-<part name="IC10" library="joakim" deviceset="DG412-J" device="T" value="DG412-JT"/>
-<part name="IC11" library="joakim" deviceset="DG412-J" device="T" value="DG412-JT"/>
+<part name="IC8" library="joakim" deviceset="DG412-J" device="S" value="DG412-JS"/>
+<part name="IC9" library="joakim" deviceset="DG412-J" device="S" value="DG412-JS"/>
+<part name="IC10" library="joakim" deviceset="DG412-J" device="S" value="DG412-JS"/>
+<part name="IC11" library="joakim" deviceset="DG412-J" device="S" value="DG412-JS"/>
 <part name="R4" library="rcl" library_urn="urn:adsk.eagle:library:334" deviceset="R-EU_" device="R0402" package3d_urn="urn:adsk.eagle:package:23547/3" value="47k"/>
 <part name="R7" library="rcl" library_urn="urn:adsk.eagle:library:334" deviceset="R-EU_" device="R0402" package3d_urn="urn:adsk.eagle:package:23547/3" value="47k"/>
@@
 <text x="-7.62" y="12.7" size="1.778" layer="97">Add to increase
 gain for noise</text>
+<text x="134.62" y="101.6" size="3.81" layer="91">SOIC16 version available as Pre-order at
+JLCPCB, half price or less than TSSOP</text>
 </plain>
 <instances>

Commit message: Rotated op amp to better suit power lines
Connections:
- net BUS_A: now also IC4C.-IN; no longer IC4A.-IN
- net BUS_B: now also IC4B.-IN; no longer IC4D.-IN
- net BUS_FX_A: now also IC4D.-IN; no longer IC4B.-IN
- net BUS_FX_B: now also IC4A.-IN; no longer IC4C.-IN
- net SUM_A: now also IC4C.OUT; no longer IC4A.OUT
- net SUM_B: now also IC4B.OUT; no longer IC4D.OUT
- net SUM_FX_A: now also IC4D.OUT; no longer IC4B.OUT
- net SUM_FX_B: now also IC4A.OUT; no longer IC4C.OUT
Other:
- moved on the sheet: IC4A, IC4B, IC4C, IC4D
Changed lines of the file:
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@@
 </instance>
 <instance part="IC2" gate="P" x="132.08" y="-167.64" smashed="yes"/>
-<instance part="IC4" gate="A" x="261.62" y="15.24" smashed="yes">
-<attribute name="NAME" x="264.16" y="18.415" size="1.778" layer="95"/>
-<attribute name="VALUE" x="264.16" y="10.16" size="1.778" layer="96"/>
-</instance>
-<instance part="IC4" gate="B" x="261.62" y="-55.88" smashed="yes">
-<attribute name="NAME" x="264.16" y="-52.705" size="1.778" layer="95"/>
-<attribute name="VALUE" x="264.16" y="-60.96" size="1.778" layer="96"/>
-</instance>
-<instance part="IC4" gate="C" x="261.62" y="-88.9" smashed="yes">
-<attribute name="NAME" x="264.16" y="-85.725" size="1.778" layer="95"/>
-<attribute name="VALUE" x="264.16" y="-93.98" size="1.778" layer="96"/>
-</instance>
-<instance part="IC4" gate="D" x="261.62" y="-17.78" smashed="yes">
-<attribute name="NAME" x="264.16" y="-14.605" size="1.778" layer="95"/>
-<attribute name="VALUE" x="264.16" y="-22.86" size="1.778" layer="96"/>
-</instance>
 <instance part="IC4" gate="P" x="134.62" y="-167.64" smashed="yes"/>
 <instance part="C23" gate="G$1" x="170.18" y="-170.18" smashed="yes" rot="R180">
@@
 <attribute name="NAME" x="123.19" y="-133.5786" size="1.778" layer="95" rot="R180"/>
 <attribute name="VALUE" x="123.19" y="-128.778" size="1.778" layer="96" rot="R180"/>
+</instance>
+<instance part="IC4" gate="A" x="261.62" y="-88.9" smashed="yes">
+<attribute name="NAME" x="264.16" y="-85.725" size="1.778" layer="95"/>
+<attribute name="VALUE" x="264.16" y="-93.98" size="1.778" layer="96"/>
+</instance>
+<instance part="IC4" gate="C" x="261.62" y="15.24" smashed="yes">
+<attribute name="NAME" x="264.16" y="18.415" size="1.778" layer="95"/>
+<attribute name="VALUE" x="264.16" y="10.16" size="1.778" layer="96"/>
+</instance>
+<instance part="IC4" gate="D" x="261.62" y="-55.88" smashed="yes">
+<attribute name="NAME" x="264.16" y="-52.705" size="1.778" layer="95"/>
+<attribute name="VALUE" x="264.16" y="-60.96" size="1.778" layer="96"/>
+</instance>
+<instance part="IC4" gate="B" x="261.62" y="-17.78" smashed="yes">
+<attribute name="NAME" x="264.16" y="-14.605" size="1.778" layer="95"/>
+<attribute name="VALUE" x="264.16" y="-22.86" size="1.778" layer="96"/>
 </instance>
 </instances>
@@
 <wire x1="251.46" y1="12.7" x2="254" y2="12.7" width="0.1524" layer="91"/>
 <pinref part="GND27" gate="1" pin="GND"/>
-<pinref part="IC4" gate="A" pin="+IN"/>
+<pinref part="IC4" gate="C" pin="+IN"/>
 </segment>
 <segment>
 <wire x1="251.46" y1="-20.32" x2="254" y2="-20.32" width="0.1524" layer="91"/>
 <pinref part="GND28" gate="1" pin="GND"/>
-<pinref part="IC4" gate="D" pin="+IN"/>
+<pinref part="IC4" gate="B" pin="+IN"/>
 </segment>
 <segment>
@@
 <wire x1="251.46" y1="-58.42" x2="254" y2="-58.42" width="0.1524" layer="91"/>
 <pinref part="GND22" gate="1" pin="GND"/>
-<pinref part="IC4" gate="B" pin="+IN"/>
+<pinref part="IC4" gate="D" pin="+IN"/>
 </segment>
 <segment>
 <wire x1="251.46" y1="-91.44" x2="254" y2="-91.44" width="0.1524" layer="91"/>
 <pinref part="GND23" gate="1" pin="GND"/>
-<pinref part="IC4" gate="C" pin="+IN"/>
+<pinref part="IC4" gate="A" pin="+IN"/>
 </segment>
 <segment>
@@
 <junction x="185.42" y="-7.62"/>
 <wire x1="185.42" y1="-15.24" x2="246.38" y2="-15.24" width="0.1524" layer="91"/>
-<pinref part="IC4" gate="D" pin="-IN"/>
 <wire x1="251.46" y1="-7.62" x2="251.46" y2="2.54" width="0.1524" layer="91"/>
 <junction x="251.46" y="-7.62"/>
 <pinref part="C25" gate="G$1" pin="1"/>
 <wire x1="251.46" y1="2.54" x2="256.54" y2="2.54" width="0.1524" layer="91"/>
+<pinref part="IC4" gate="B" pin="-IN"/>
 </segment>
 </net>
@@
 <wire x1="175.26" y1="-12.7" x2="220.98" y2="-12.7" width="0.1524" layer="91"/>
 <wire x1="220.98" y1="-12.7" x2="220.98" y2="17.78" width="0.1524" layer="91"/>
-<pinref part="IC4" gate="A" pin="-IN"/>
 <wire x1="251.46" y1="25.4" x2="251.46" y2="35.56" width="0.1524" layer="91"/>
 <junction x="251.46" y="25.4"/>
 <pinref part="C24" gate="G$1" pin="1"/>
 <wire x1="251.46" y1="35.56" x2="256.54" y2="35.56" width="0.1524" layer="91"/>
+<pinref part="IC4" gate="C" pin="-IN"/>
 </segment>
 </net>
@@
 <label x="274.32" y="15.24" size="1.778" layer="95"/>
 <wire x1="271.78" y1="15.24" x2="287.02" y2="15.24" width="0.1524" layer="91"/>
-<pinref part="IC4" gate="A" pin="OUT"/>
 <pinref part="C24" gate="G$1" pin="2"/>
 <wire x1="264.16" y1="35.56" x2="271.78" y2="35.56" width="0.1524" layer="91"/>
 <wire x1="271.78" y1="35.56" x2="271.78" y2="25.4" width="0.1524" layer="91"/>
 <junction x="271.78" y="25.4"/>
+<pinref part="IC4" gate="C" pin="OUT"/>
 </segment>
 <segment>
@@
 <label x="274.32" y="-17.78" size="1.778" layer="95"/>
 <wire x1="271.78" y1="-17.78" x2="287.02" y2="-17.78" width="0.1524" layer="91"/>
-<pinref part="IC4" gate="D" pin="OUT"/>
 <pinref part="C25" gate="G$1" pin="2"/>
 <wire x1="264.16" y1="2.54" x2="271.78" y2="2.54" width="0.1524" layer="91"/>
 <wire x1="271.78" y1="2.54" x2="271.78" y2="-7.62" width="0.1524" layer="91"/>
 <junction x="271.78" y="-7.62"/>
+<pinref part="IC4" gate="B" pin="OUT"/>
 </segment>
 <segment>
@@
 <label x="274.32" y="-88.9" size="1.778" layer="95"/>
 <wire x1="271.78" y1="-88.9" x2="287.02" y2="-88.9" width="0.1524" layer="91"/>
-<pinref part="IC4" gate="C" pin="OUT"/>
 <pinref part="C27" gate="G$1" pin="2"/>
 <wire x1="264.16" y1="-68.58" x2="271.78" y2="-68.58" width="0.1524" layer="91"/>
 <wire x1="271.78" y1="-68.58" x2="271.78" y2="-78.74" width="0.1524" layer="91"/>
 <junction x="271.78" y="-78.74"/>
+<pinref part="IC4" gate="A" pin="OUT"/>
 </segment>
 <segment>
@@
 <label x="274.32" y="-55.88" size="1.778" layer="95"/>
 <wire x1="271.78" y1="-55.88" x2="287.02" y2="-55.88" width="0.1524" layer="91"/>
-<pinref part="IC4" gate="B" pin="OUT"/>
 <pinref part="C26" gate="G$1" pin="2"/>
 <wire x1="264.16" y1="-35.56" x2="271.78" y2="-35.56" width="0.1524" layer="91"/>
 <wire x1="271.78" y1="-35.56" x2="271.78" y2="-45.72" width="0.1524" layer="91"/>
 <junction x="271.78" y="-45.72"/>
+<pinref part="IC4" gate="D" pin="OUT"/>
 </segment>
 <segment>
@@
 <wire x1="246.38" y1="-58.42" x2="246.38" y2="-53.34" width="0.1524" layer="91"/>
 <junction x="246.38" y="-53.34"/>
-<pinref part="IC4" gate="B" pin="-IN"/>
 <wire x1="251.46" y1="-45.72" x2="251.46" y2="-35.56" width="0.1524" layer="91"/>
 <junction x="251.46" y="-45.72"/>
 <pinref part="C26" gate="G$1" pin="1"/>
 <wire x1="251.46" y1="-35.56" x2="256.54" y2="-35.56" width="0.1524" layer="91"/>
+<pinref part="IC4" gate="D" pin="-IN"/>
 </segment>
 </net>
@@
 <wire x1="185.42" y1="-48.26" x2="185.42" y2="-86.36" width="0.1524" layer="91"/>
 <wire x1="185.42" y1="-86.36" x2="246.38" y2="-86.36" width="0.1524" layer="91"/>
-<pinref part="IC4" gate="C" pin="-IN"/>
 <wire x1="251.46" y1="-78.74" x2="251.46" y2="-68.58" width="0.1524" layer="91"/>
 <junction x="251.46" y="-78.74"/>
 <pinref part="C27" gate="G$1" pin="1"/>
 <wire x1="251.46" y1="-68.58" x2="256.54" y2="-68.58" width="0.1524" layer="91"/>
-</segment>
-</net>
+<pinref part="IC4" gate="A" pin="-IN"/>
+</segment>
+</net>

Commit message: Everything but fuckup-protection-resistor routed
Connections:
- net DIG_1_BUS_B: now also R93.2; no longer R83.2
- net DIG_2_BUS_A: now also R83.2; no longer R84.2
- net DIG_2_BUS_B: now also R92.2; no longer R85.2
- net DIG_3_BUS_A: now also R84.2; no longer R94.2
- net DIG_3_BUS_B: now also R90.2; no longer R95.2
- net DIG_4_BUS_A: now also R85.2; no longer R96.2
- net DIG_4_BUS_B: now also R91.2; no longer R97.2
- net DIG_5_BUS_A: now also R94.2; no longer R92.2
- net DIG_5_BUS_B: now also R86.2; no longer R93.2
- net DIG_6_BUS_A: now also R95.2; no longer R90.2
- net DIG_6_BUS_B: now also R87.2; no longer R91.2
- net DIG_7_BUS_A: now also R96.2; no longer R86.2
- net DIG_7_BUS_B: now also R88.2; no longer R87.2
- net DIG_8_BUS_A: now also R97.2; no longer R88.2
Changed lines of the file:
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@@
 </segment>
 <segment>
-<label x="246.38" y="-147.32" size="1.778" layer="95"/>
-<wire x1="264.16" y1="-147.32" x2="241.3" y2="-147.32" width="0.1524" layer="91"/>
-<pinref part="R84" gate="G$1" pin="2"/>
+<label x="246.38" y="-144.78" size="1.778" layer="95"/>
+<wire x1="264.16" y1="-144.78" x2="241.3" y2="-144.78" width="0.1524" layer="91"/>
+<pinref part="R83" gate="G$1" pin="2"/>
 </segment>
 </net>
@@
 </segment>
 <segment>
-<label x="246.38" y="-149.86" size="1.778" layer="95"/>
-<wire x1="264.16" y1="-149.86" x2="241.3" y2="-149.86" width="0.1524" layer="91"/>
-<pinref part="R85" gate="G$1" pin="2"/>
+<label x="246.38" y="-170.18" size="1.778" layer="95"/>
+<wire x1="264.16" y1="-170.18" x2="241.3" y2="-170.18" width="0.1524" layer="91"/>
+<pinref part="R92" gate="G$1" pin="2"/>
 </segment>
 </net>
@@
 </segment>
 <segment>
-<label x="246.38" y="-177.8" size="1.778" layer="95"/>
-<wire x1="264.16" y1="-177.8" x2="241.3" y2="-177.8" width="0.1524" layer="91"/>
-<pinref part="R95" gate="G$1" pin="2"/>
+<label x="246.38" y="-165.1" size="1.778" layer="95"/>
+<wire x1="264.16" y1="-165.1" x2="241.3" y2="-165.1" width="0.1524" layer="91"/>
+<pinref part="R90" gate="G$1" pin="2"/>
 </segment>
 </net>
@@
 </segment>
 <segment>
-<label x="246.38" y="-175.26" size="1.778" layer="95"/>
-<wire x1="264.16" y1="-175.26" x2="241.3" y2="-175.26" width="0.1524" layer="91"/>
-<pinref part="R94" gate="G$1" pin="2"/>
+<label x="246.38" y="-147.32" size="1.778" layer="95"/>
+<wire x1="264.16" y1="-147.32" x2="241.3" y2="-147.32" width="0.1524" layer="91"/>
+<pinref part="R84" gate="G$1" pin="2"/>
 </segment>
 </net>
@@
 </segment>
 <segment>
-<label x="246.38" y="-144.78" size="1.778" layer="95"/>
-<wire x1="264.16" y1="-144.78" x2="241.3" y2="-144.78" width="0.1524" layer="91"/>
-<pinref part="R83" gate="G$1" pin="2"/>
+<label x="246.38" y="-172.72" size="1.778" layer="95"/>
+<wire x1="264.16" y1="-172.72" x2="241.3" y2="-172.72" width="0.1524" layer="91"/>
+<pinref part="R93" gate="G$1" pin="2"/>
 </segment>
 </net>
@@
 </segment>
 <segment>
-<label x="246.38" y="-182.88" size="1.778" layer="95"/>
-<wire x1="264.16" y1="-182.88" x2="241.3" y2="-182.88" width="0.1524" layer="91"/>
-<pinref part="R97" gate="G$1" pin="2"/>
+<label x="246.38" y="-167.64" size="1.778" layer="95"/>
+<wire x1="264.16" y1="-167.64" x2="241.3" y2="-167.64" width="0.1524" layer="91"/>
+<pinref part="R91" gate="G$1" pin="2"/>
 </segment>
 </net>
@@
 </segment>
 <segment>
-<label x="246.38" y="-180.34" size="1.778" layer="95"/>
-<wire x1="264.16" y1="-180.34" x2="241.3" y2="-180.34" width="0.1524" layer="91"/>
-<pinref part="R96" gate="G$1" pin="2"/>
+<label x="246.38" y="-149.86" size="1.778" layer="95"/>
+<wire x1="264.16" y1="-149.86" x2="241.3" y2="-149.86" width="0.1524" layer="91"/>
+<pinref part="R85" gate="G$1" pin="2"/>
 </segment>
 </net>
@@
 </segment>
 <segment>
-<label x="246.38" y="-172.72" size="1.778" layer="95"/>
-<wire x1="264.16" y1="-172.72" x2="241.3" y2="-172.72" width="0.1524" layer="91"/>
-<pinref part="R93" gate="G$1" pin="2"/>
+<label x="246.38" y="-152.4" size="1.778" layer="95"/>
+<wire x1="264.16" y1="-152.4" x2="241.3" y2="-152.4" width="0.1524" layer="91"/>
+<pinref part="R86" gate="G$1" pin="2"/>
 </segment>
 </net>
@@
 </segment>
 <segment>
-<label x="246.38" y="-170.18" size="1.778" layer="95"/>
-<wire x1="264.16" y1="-170.18" x2="241.3" y2="-170.18" width="0.1524" layer="91"/>
-<pinref part="R92" gate="G$1" pin="2"/>
+<label x="246.38" y="-175.26" size="1.778" layer="95"/>
+<wire x1="264.16" y1="-175.26" x2="241.3" y2="-175.26" width="0.1524" layer="91"/>
+<pinref part="R94" gate="G$1" pin="2"/>
 </segment>
 </net>
@@
 </segment>
 <segment>
-<label x="246.38" y="-167.64" size="1.778" layer="95"/>
-<wire x1="264.16" y1="-167.64" x2="241.3" y2="-167.64" width="0.1524" layer="91"/>
-<pinref part="R91" gate="G$1" pin="2"/>
+<label x="246.38" y="-154.94" size="1.778" layer="95"/>
+<wire x1="264.16" y1="-154.94" x2="241.3" y2="-154.94" width="0.1524" layer="91"/>
+<pinref part="R87" gate="G$1" pin="2"/>
 </segment>
 </net>
@@
 </segment>
 <segment>
-<label x="246.38" y="-165.1" size="1.778" layer="95"/>
-<wire x1="264.16" y1="-165.1" x2="241.3" y2="-165.1" width="0.1524" layer="91"/>
-<pinref part="R90" gate="G$1" pin="2"/>
+<label x="246.38" y="-177.8" size="1.778" layer="95"/>
+<wire x1="264.16" y1="-177.8" x2="241.3" y2="-177.8" width="0.1524" layer="91"/>
+<pinref part="R95" gate="G$1" pin="2"/>
 </segment>
 </net>
@@
 </segment>
 <segment>
-<label x="246.38" y="-152.4" size="1.778" layer="95"/>
-<wire x1="264.16" y1="-152.4" x2="241.3" y2="-152.4" width="0.1524" layer="91"/>
-<pinref part="R86" gate="G$1" pin="2"/>
+<label x="246.38" y="-180.34" size="1.778" layer="95"/>
+<wire x1="264.16" y1="-180.34" x2="241.3" y2="-180.34" width="0.1524" layer="91"/>
+<pinref part="R96" gate="G$1" pin="2"/>
 </segment>
 </net>
@@
 </segment>
 <segment>
-<label x="246.38" y="-154.94" size="1.778" layer="95"/>
-<wire x1="264.16" y1="-154.94" x2="241.3" y2="-154.94" width="0.1524" layer="91"/>
-<pinref part="R87" gate="G$1" pin="2"/>
+<label x="246.38" y="-157.48" size="1.778" layer="95"/>
+<wire x1="264.16" y1="-157.48" x2="241.3" y2="-157.48" width="0.1524" layer="91"/>
+<pinref part="R88" gate="G$1" pin="2"/>
 </segment>
 </net>
@@
 </segment>
 <segment>
-<label x="246.38" y="-157.48" size="1.778" layer="95"/>
-<wire x1="264.16" y1="-157.48" x2="241.3" y2="-157.48" width="0.1524" layer="91"/>
-<pinref part="R88" gate="G$1" pin="2"/>
+<label x="246.38" y="-182.88" size="1.778" layer="95"/>
+<wire x1="264.16" y1="-182.88" x2="241.3" y2="-182.88" width="0.1524" layer="91"/>
+<pinref part="R97" gate="G$1" pin="2"/>
 </segment>
 </net>

Commit message: Finished except perhaps holes and DNM resistor for noise gain
Other:
- note added: "R70 - noise gain: Decide value before ordering instead of having this."
- note removed: "1.2: 2 x 16p instead of 1 x 32p 1.3: ext input to output B, to add SVF output, mixed here to get clipping BEFORE Juno filter 1.4: Error in out b gain, was double. Also added attenuation of input to prevent clipping in filter"
Changed lines of the file:
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@@
 is inv
 here</text>
-<text x="-152.4" y="78.74" size="3.81" layer="91">1.2: 2 x 16p instead of 1 x 32p
-1.3: ext input to output B, to add
-SVF output, mixed here to get clipping BEFORE
-Juno filter
-1.4: Error in out b gain, was double. Also added
-attenuation of input to prevent
-clipping in filter</text>
+<text x="-152.4" y="78.74" size="3.81" layer="91">R70 - noise gain: Decide value before
+ordering instead of having this.</text>
 <text x="106.68" y="-66.04" size="1.778" layer="91">NB: SVF Chain
 is inverting!</text>
 <text x="-7.62" y="12.7" size="1.778" layer="97">Add to increase
 gain for noise</text>
-<text x="134.62" y="101.6" size="3.81" layer="91">SOIC16 version available as Pre-order at
+<text x="-152.4" y="96.52" size="3.81" layer="91">SOIC16 version available as Pre-order at
 JLCPCB, half price or less than TSSOP</text>
 </plain>
