File: Bus_Mixer/export-v7.7/AS3364_DG412_bus_mixer_v1.3.brd (EAGLE design)
At the start: 84.8 x 52.5 mm, 124 parts, among them IC1 PCA9539PW, IC10 DG412-J, IC11 DG412-J, IC2 TL074JT, IC3 TL072JT, IC4 TL074JT, IC6 TL072JT, IC7 TL074JT, IC8 DG412-J, IC9 DG412-J

Commit message: export v7
Parts:
- removed IC7: TL074JT, joakim:TSSOP14J
- removed R71: 47k, rcl:R0402
- added IC5: TL072JT, joakim:TSSOP8J
- R28, R31, R34, R37: value 100k -> 47k
- moved R51 10.00 mm to (41.9, 8.73), turned to 270 degrees
- moved R43 0.65 mm to (29.4, 19.2)
Connections:
- removed net N$20: IC7.14, R51.1, R71.2
- removed net N$22: IC7.1, IC7.2
- net +12V: now also IC5.8; no longer IC7.4
- net -12V: now also IC5.4; no longer IC7.11
- net CON3: now also IC5.6; no longer IC7.6
- net CON4: now also IC5.2; no longer IC7.9
- net GND: now also IC5.3, IC5.5, R51.2; no longer IC2.10, IC7.10, IC7.12, IC7.3, IC7.5
- net N$17: now also IC2.10, R51.1; no longer IC7.13, R51.2
- net N$6: no longer R71.1
- net OUT3: now also IC5.7; no longer IC7.7
- net OUT4: now also IC5.1; no longer IC7.8
Routing:
- net N$20: track 15.0 -> 0.00 mm, vias 2 -> 0
- net OUT3: track 18.1 -> 24.1 mm
- net N$6: track 21.2 -> 16.3 mm
- net N$17: track 14.5 -> 18.1 mm
- net OUT4: track 31.5 -> 33.1 mm
- net CON4: track 15.9 -> 14.9 mm
- net N$22: track 0.65 -> 0.00 mm
- net CV_A_DRY: vias 1 -> 0
Other:
- outline, holes or cut-outs redrawn
- board text added: "Pre-filter bus mixer DG412 version v1.3"
- board text removed: "Pre-filter bus mixer DG412 version v1.4"
