File: Bus_Mixer/export-v7.7/AS3364_DG412_bus_mixer_v1.3.sch (EAGLE design)
At the start: 123 parts, among them IC1 PCA9539PW, IC10 DG412-J, IC11 DG412-J, IC2 TL074JT, IC3 TL072JT, IC4 TL074JT, IC6 TL072JT, IC7 TL074JT, IC8 DG412-J, IC9 DG412-J

Commit message: export v7
Parts:
- removed IC7: TL074JT, joakim:TL074JT
- removed R71: 47k, rcl:R-EU_R0402
- added IC5: TL072JT, joakim:TL072JT
- R28, R31, R34, R37: value 100k -> 47k
Connections:
- removed net N$20: IC7D.OUT, R51.1, R71.2
- removed net N$22: IC7A.-IN, IC7A.OUT
- net +12V: now also IC5P.V+; no longer IC7P.V+
- net -12V: now also IC5P.V-; no longer IC7P.V-
- net CON3: now also IC5B.-IN; no longer IC7B.-IN
- net CON4: now also IC5A.-IN; no longer IC7C.-IN
- net GND: now also IC5A.+IN, IC5B.+IN, R51.2; no longer IC2C.+IN, IC7A.+IN, IC7B.+IN, IC7C.+IN, IC7D.+IN
- net N$17: now also IC2C.+IN, R51.1; no longer IC7D.-IN, R51.2
- net N$6: no longer R71.1
- net OUT3: now also IC5B.OUT; no longer IC7B.OUT
- net OUT4: now also IC5A.OUT; no longer IC7C.OUT
Other:
- note added: "1.2: 2 x 16p instead of 1 x 32p 1.3: ext input to output B, to add SVF output, mixed here to get clipping BEFORE Juno filter"
- note added: "Funker finfint!"
- note added: "Inverts FX but not Dry so output is in phase"
- note removed: "1.2: 2 x 16p instead of 1 x 32p 1.3: ext input to output B, to add SVF output, mixed here to get clipping BEFORE Juno filter 1.4: Error in out b gain, was double. Also added attenuation of input to prevent clipping in filter"
- note removed: "TODO: Bruke opamp 2 til å invertere DRY A?"
- moved on the sheet: IC2C, R50, R51, R69
